Commit message: update much more

File: src/carver_description/urdf/carver.urdf.xacro (robot description, xacro)
@@ -4,5 +4,8 @@
   <xacro:include filename="$(find carver_description)/urdf/gazebo_control.xacro" />
   <xacro:include filename="$(find carver_description)/urdf/inertial_macros.xacro" />
-  <link
+  <xacro:include filename="$(find carver_description)/urdf/imu.xacro" />
+  <xacro:include filename="$(find carver_description)/urdf/laser.xacro" />
+  <xacro:include filename="$(find carver_description)/urdf/gps.xacro" />
+<link
     name="base_link">
     <inertial>
@@ -26,19 +29,19 @@
       <geometry>
         <mesh
-          filename="file://$(find carver_description)/meshes/base_link.dae" />
-      </geometry>
-      <material
-        name="">
-        <color
-          rgba="0.792156862745098 0.819607843137255 0.933333333333333 1" />
-      </material>
-    </visual>
-    <collision>
-      <origin
-        xyz="0 0 0"
-        rpy="0 0 0" />
-      <geometry>
-        <mesh
-          filename="file://$(find carver_description)/meshes/base_link.dae" />
+          filename="file://$(find carver_description)/meshes/base_link.STL" />
+      </geometry>
+      <material
+        name="">
+        <color
+          rgba="0.792156862745098 0.819607843137255 0.933333333333333 1" />
+      </material>
+    </visual>
+    <collision>
+      <origin
+        xyz="0 0 0"
+        rpy="0 0 0" />
+      <geometry>
+        <mesh
+          filename="file://$(find carver_description)/meshes/base_link.STL" />
       </geometry>
     </collision>
@@ -57,7 +60,6 @@
         rpy="0 0 0" />
       <mass
-        value="0.25" />
-      <inertia ixx="0.00525" ixy="0" ixz="0" iyy="0.00035" iyz="0" izz="0.00525" />
-      <!-- <inertia
+        value="0.0307417074716638" />
+      <inertia
         ixx="5.15827058483555E-06"
         ixy="2.87694711205719E-08"
@@ -65,27 +67,27 @@
         iyy="5.94711293506547E-06"
         iyz="1.79592218418332E-13"
-        izz="8.17709432093611E-06" /> -->
-    </inertial>
-    <visual>
-      <origin
-        xyz="0 0 0"
-        rpy="0 0 0" />
-      <geometry>
-        <mesh
-          filename="file://$(find carver_description)/meshes/front_right_sterring_Link.dae" />
-      </geometry>
-      <material
-        name="">
-        <color
-          rgba="0.792156862745098 0.819607843137255 0.933333333333333 1" />
-      </material>
-    </visual>
-    <collision>
-      <origin
-        xyz="0 0 0"
-        rpy="0 0 0" />
-      <geometry>
-        <mesh
-          filename="file://$(find carver_description)/meshes/front_right_sterring_Link.dae" />
+        izz="8.17709432093611E-06" />
+    </inertial>
+    <visual>
+      <origin
+        xyz="0 0 0"
+        rpy="0 0 0" />
+      <geometry>
+        <mesh
+          filename="file://$(find carver_description)/meshes/front_right_sterring_Link.STL" />
+      </geometry>
+      <material
+        name="">
+        <color
+          rgba="0.792156862745098 0.819607843137255 0.933333333333333 1" />
+      </material>
+    </visual>
+    <collision>
+      <origin
+        xyz="0 0 0"
+        rpy="0 0 0" />
+      <geometry>
+        <mesh
+          filename="file://$(find carver_description)/meshes/front_right_sterring_Link.STL" />
       </geometry>
     </collision>
@@ -104,8 +106,8 @@
       xyz="0 0 -1" />
     <limit
-      lower="-0.698132"
-      upper="0.698132"
-      effort="1000"
-      velocity="1.0" />
+      lower="-3.14"
+      upper="3.14"
+      effort="100"
+      velocity="100" />
   </joint>
   <link
@@ -131,19 +133,19 @@
       <geometry>
         <mesh
-          filename="file://$(find carver_description)/meshes/front_right_wheel_Link.dae" />
-      </geometry>
-      <material
-        name="">
-        <color
-          rgba="0.792156862745098 0.819607843137255 0.933333333333333 1" />
-      </material>
-    </visual>
-    <collision>
-      <origin
-        xyz="0 0 0"
-        rpy="0 0 0" />
-      <geometry>
-        <mesh
-          filename="file://$(find carver_description)/meshes/front_right_wheel_Link.dae" />
+          filename="file://$(find carver_description)/meshes/front_right_wheel_Link.STL" />
+      </geometry>
+      <material
+        name="">
+        <color
+          rgba="0.792156862745098 0.819607843137255 0.933333333333333 1" />
+      </material>
+    </visual>
+    <collision>
+      <origin
+        xyz="0 0 0"
+        rpy="0 0 0" />
+      <geometry>
+        <mesh
+          filename="file://$(find carver_description)/meshes/front_right_wheel_Link.STL" />
       </geometry>
     </collision>
@@ -172,7 +174,6 @@
         rpy="0 0 0" />
       <mass
-        value="0.25" />
-      <inertia ixx="0.00525" ixy="0" ixz="0" iyy="0.00035" iyz="0" izz="0.00525" />
-      <!-- <inertia
+        value="0.0307417074716638" />
+      <inertia
         ixx="5.15827283476504E-06"
         ixy="-2.88003004005144E-08"
@@ -180,27 +181,27 @@
         iyy="5.94711068513598E-06"
         iyz="-6.03807311086712E-15"
-        izz="8.17709432093612E-06" /> -->
-    </inertial>
-    <visual>
-      <origin
-        xyz="0 0 0"
-        rpy="0 0 0" />
-      <geometry>
-        <mesh
-          filename="file://$(find carver_description)/meshes/front_left_sterring_Link.dae" />
-      </geometry>
-      <material
-        name="">
-        <color
-          rgba="0.792156862745098 0.819607843137255 0.933333333333333 1" />
-      </material>
-    </visual>
-    <collision>
-      <origin
-        xyz="0 0 0"
-        rpy="0 0 0" />
-      <geometry>
-        <mesh
-          filename="file://$(find carver_description)/meshes/front_left_sterring_Link.dae" />
+        izz="8.17709432093612E-06" />
+    </inertial>
+    <visual>
+      <origin
+        xyz="0 0 0"
+        rpy="0 0 0" />
+      <geometry>
+        <mesh
+          filename="file://$(find carver_description)/meshes/front_left_sterring_Link.STL" />
+      </geometry>
+      <material
+        name="">
+        <color
+          rgba="0.792156862745098 0.819607843137255 0.933333333333333 1" />
+      </material>
+    </visual>
+    <collision>
+      <origin
+        xyz="0 0 0"
+        rpy="0 0 0" />
+      <geometry>
+        <mesh
+          filename="file://$(find carver_description)/meshes/front_left_sterring_Link.STL" />
       </geometry>
     </collision>
@@ -219,8 +220,8 @@
       xyz="0 0 -1" />
     <limit
-      lower="-0.698132"
-      upper="0.698132"
-      effort="1000"
-      velocity="1.0" />
+      lower="-3.14"
+      upper="3.14"
+      effort="100"
+      velocity="100" />
   </joint>
   <link
@@ -246,19 +247,19 @@
       <geometry>
         <mesh
-          filename="file://$(find carver_description)/meshes/front_left_wheel_Link.dae" />
-      </geometry>
-      <material
-        name="">
-        <color
-          rgba="0.792156862745098 0.819607843137255 0.933333333333333 1" />
-      </material>
-    </visual>
-    <collision>
-      <origin
-        xyz="0 0 0"
-        rpy="0 0 0" />
-      <geometry>
-        <mesh
-          filename="file://$(find carver_description)/meshes/front_left_wheel_Link.dae" />
+          filename="file://$(find carver_description)/meshes/front_left_wheel_Link.STL" />
+      </geometry>
+      <material
+        name="">
+        <color
+          rgba="0.792156862745098 0.819607843137255 0.933333333333333 1" />
+      </material>
+    </visual>
+    <collision>
+      <origin
+        xyz="0 0 0"
+        rpy="0 0 0" />
+      <geometry>
+        <mesh
+          filename="file://$(find carver_description)/meshes/front_left_wheel_Link.STL" />
       </geometry>
     </collision>
@@ -302,19 +303,19 @@
       <geometry>
         <mesh
-          filename="file://$(find carver_description)/meshes/rear_right_wheel_Link.dae" />
-      </geometry>
-      <material
-        name="">
-        <color
-          rgba="0.792156862745098 0.819607843137255 0.933333333333333 1" />
-      </material>
-    </visual>
-    <collision>
-      <origin
-        xyz="0 0 0"
-        rpy="0 0 0" />
-      <geometry>
-        <mesh
-          filename="file://$(find carver_description)/meshes/rear_right_wheel_Link.dae" />
+          filename="file://$(find carver_description)/meshes/rear_right_wheel_Link.STL" />
+      </geometry>
+      <material
+        name="">
+        <color
+          rgba="0.792156862745098 0.819607843137255 0.933333333333333 1" />
+      </material>
+    </visual>
+    <collision>
+      <origin
+        xyz="0 0 0"
+        rpy="0 0 0" />
+      <geometry>
+        <mesh
+          filename="file://$(find carver_description)/meshes/rear_right_wheel_Link.STL" />
       </geometry>
     </collision>
@@ -334,5 +335,5 @@
     <limit
       effort="100"
-      velocity="10" />
+      velocity="100" />
   </joint>
   <link
@@ -358,19 +359,19 @@
       <geometry>
         <mesh
-          filename="file://$(find carver_description)/meshes/rear_left_wheel_Link.dae" />
-      </geometry>
-      <material
-        name="">
-        <color
-          rgba="0.792156862745098 0.819607843137255 0.933333333333333 1" />
-      </material>
-    </visual>
-    <collision>
-      <origin
-        xyz="0 0 0"
-        rpy="0 0 0" />
-      <geometry>
-        <mesh
-          filename="file://$(find carver_description)/meshes/rear_left_wheel_Link.dae" />
+          filename="file://$(find carver_description)/meshes/rear_left_wheel_Link.STL" />
+      </geometry>
+      <material
+        name="">
+        <color
+          rgba="0.792156862745098 0.819607843137255 0.933333333333333 1" />
+      </material>
+    </visual>
+    <collision>
+      <origin
+        xyz="0 0 0"
+        rpy="0 0 0" />
+      <geometry>
+        <mesh
+          filename="file://$(find carver_description)/meshes/rear_left_wheel_Link.STL" />
       </geometry>
     </collision>
@@ -390,5 +391,5 @@
     <limit
       effort="100"
-      velocity="10" />
+      velocity="100" />
   </joint>
   <link
@@ -604,6 +605,5 @@
       xyz="0 0 0" />
   </joint>
-<!-- /////////////////////////////// -->
-  <link name="laser"></link>
+  <!-- <link name="laser"></link>
   <joint name="base_laser_joint" type="fixed">
     <parent link="base_link"/>
@@ -611,5 +611,4 @@
     <origin xyz="0 0 0.154015" rpy="0 0 0"/>
   </joint>
-<!-- /////////////////////////////// -->
   <link
     name="RPLIDAR_LB_Link">
@@ -652,5 +651,4 @@
     </collision>
   </link>
-<!-- /////////////////////////////// -->
   <joint
     name="laser_RPLIDAR_LB_joint"
@@ -666,5 +664,4 @@
       xyz="0 0 0" />
   </joint>
-<!-- /////////////////////////////// -->
   <link
     name="IMU_R_Link">
@@ -813,5 +810,4 @@
     </collision>
   </link>
-<!-- /////////////////////////////// -->
   <joint
     name="laser_RPLIDAR_RF_joint"
@@ -827,5 +823,4 @@
       xyz="0 0 0" />
   </joint>
-<!-- /////////////////////////////// -->
   <link
     name="GPS_Link">
@@ -880,4 +875,4 @@
     <axis
       xyz="0 0 0" />
-  </joint>
+  </joint> -->
 </robot>

File: src/carver_description/urdf/gazebo.xacro (robot description, xacro)
@@ -25,3 +25,140 @@
         </transmission>
   </xacro:macro>
+    <xacro:macro name="gazebo_laser" params="frame_prefix">
+        <gazebo reference="${frame_prefix}_link">
+            <sensor name="laser" type="ray">
+            <always_on>true</always_on>
+            <visualize>false</visualize>
+            <update_rate>10</update_rate>
+            <ray>
+                <scan>
+                <horizontal>
+                    <samples>120</samples>
+                    <resolution>1.000000</resolution>
+                    <min_angle>-3.14159</min_angle>
+                    <max_angle>3.14159</max_angle>
+                </horizontal>
+                </scan>
+                <range>
+                <min>0.3</min>
+                <max>15.0</max>
+                <resolution>0.015</resolution>
+                </range>
+                <noise>
+                <type>gaussian</type>
+                <mean>0.0</mean>
+                <stddev>0.01</stddev>
+                </noise>
+            </ray>
+            <plugin name="scan" filename="libgazebo_ros_ray_sensor.so">
+                <ros>
+                <remapping>~/out:=scan</remapping>
+                </ros>
+                <output_type>sensor_msgs/LaserScan</output_type>
+                <frame_name>laser</frame_name>
+            </plugin>
+            </sensor>
+        </gazebo>
+    </xacro:macro>
+    <xacro:macro name="gazebo_imu" params="link_name topic frame_name">
+    <gazebo reference="${link_name}">
+        <gravity>true</gravity>
+        <sensor name="${link_name}_imu" type="imu">
+        <always_on>true</always_on>
+        <update_rate>100</update_rate>
+        <visualize>true</visualize>
+        <imu>
+            <orientation>
+            <x>
+                <noise type="gaussian">
+                <mean>0.0</mean>
+                <stddev>2e-3</stddev>
+                </noise>
+            </x>
+            <y>
+                <noise type="gaussian">
+                <mean>0.0</mean>
+                <stddev>2e-3</stddev>
+                </noise>
+            </y>
+            <z>
+                <noise type="gaussian">
+                <mean>0.0</mean>
+                <stddev>2e-3</stddev>
+                </noise>
+            </z>
+            </orientation>
+            <angular_velocity>
+            <x>
+                <noise type="gaussian">
+                <mean>0.0</mean>
+                <stddev>2e-4</stddev>
+                </noise>
+            </x>
+            <y>
+                <noise type="gaussian">
+                <mean>0.0</mean>
+                <stddev>2e-4</stddev>
+                </noise>
+            </y>
+            <z>
+                <noise type="gaussian">
+                <mean>0.0</mean>
+                <stddev>2e-4</stddev>
+                </noise>
+            </z>
+            </angular_velocity>
+            <linear_acceleration>
+            <x>
+                <noise type="gaussian">
+                <mean>0.0</mean>
+                <stddev>1.7e-2</stddev>
+                </noise>
+            </x>
+            <y>
+                <noise type="gaussian">
+                <mean>0.0</mean>
+                <stddev>1.7e-2</stddev>
+                </noise>
+            </y>
+            <z>
+                <noise type="gaussian">
+                <mean>0.0</mean>
+                <stddev>1.7e-2</stddev>
+                </noise>
+            </z>
+            </linear_acceleration>
+        </imu>
+        <plugin name="two_wheeled_robot_imu" filename="libgazebo_ros_imu_sensor.so">
+            <initial_orientation_as_reference>false</initial_orientation_as_reference>
+            <frame_name>${frame_name}_imu_link</frame_name>
+            <ros>
+            <remapping>~/out:=${topic}/imu</remapping>
+            </ros>
+        </plugin>
+        </sensor>
+    </gazebo>
+    </xacro:macro>
+    <xacro:macro name="gazebo_gps" params="link_name topic frame_name">
+    <gazebo reference="${link_name}">
+        <gravity>true</gravity>
+        <sensor name="${link_name}_gps" type="gps">
+        <always_on>true</always_on>
+        <update_rate>5</update_rate>
+        <visualize>true</visualize>
+        <pose>0 0 0 0 0 0</pose>
+        <gps>
+            <!-- Adjust smoothing or add noise parameters as required -->
+            <position_smoothing>0.5</position_smoothing>
+        </gps>
+        <plugin name="gazebo_ros_gps_sensor" filename="libgazebo_ros_gps_plugin.so">
+            <ros>
+            <remapping>~/out:=${topic}</remapping>
+            </ros>
+            <topicName>${topic}</topicName>
+            <frameName>${frame_name}</frameName>
+        </plugin>
+        </sensor>
+    </gazebo>
+    </xacro:macro>
 </robot>

File: src/carver_description/urdf/gazebo_control.xacro (robot description, xacro)
@@ -48,10 +48,14 @@
   <xacro:include filename="$(find carver_description)/urdf/gazebo.xacro" />
   <!-- Actuator configurations -->
-  <!-- <xacro:carver_wheel_transmission wheel_prefix="front_left_steering_front_right" />
+  <xacro:carver_wheel_transmission wheel_prefix="front_left_steering_front_right" />
   <xacro:carver_wheel_transmission wheel_prefix="front_left_steering_front_left" />
   <xacro:carver_wheel_transmission wheel_prefix="base_rear_left" />
   <xacro:carver_wheel_transmission wheel_prefix="base_rear_right" />
   <xacro:carver_steering_hinge_transmission wheel_prefix="base_front_right" />
-  <xacro:carver_steering_hinge_transmission wheel_prefix="base_front_left" /> -->
+  <xacro:carver_steering_hinge_transmission wheel_prefix="base_front_left" />
+  <!-- <xacro:gazebo_laser frame_prefix="laser" /> -->
+  <!-- <xacro:gazebo_imu link_name="IMU_R_Link" topic="/imu_right" frame_name="IMU_R_Link" />
+  <xacro:gazebo_imu link_name="IMU_L_Link" topic="/imu_left" frame_name="IMU_L_Link" /> -->
+  <!-- <xacro:gazebo_gps link_name="GPS_Link" topic="/gps/fix" frame_name="GPS_Link" /> -->
   <!-- Gazebo friction/contact parameters -->
   <gazebo>

Commit message: fix wheel and add laser scan sensor

File: src/carver_description/urdf/carver.urdf.xacro (robot description, xacro)
@@ -59,5 +59,5 @@
         xyz="-6.87012402522669E-09 3.51066137271872E-09 -0.0112499999237069"
         rpy="0 0 0" />
-      <mass
+      <!-- <mass
         value="0.0307417074716638" />
       <inertia
@@ -67,5 +67,7 @@
         iyy="5.94711293506547E-06"
         iyz="1.79592218418332E-13"
-        izz="8.17709432093611E-06" />
+        izz="8.17709432093611E-06" /> -->
+        <mass value="0.25" />
+        <inertia ixx="0.00525" ixy="0" ixz="0" iyy="0.00035" iyz="0" izz="0.00525" />
     </inertial>
     <visual>
@@ -97,5 +99,5 @@
     type="revolute">
     <origin
-      xyz="0.639118924633511 -0.284499999999994 -0.158749999999999"
+      xyz="0.639118924633511 -0.284499999999994 -0.17"
       rpy="0 0 0" />
     <parent
@@ -105,9 +107,5 @@
     <axis
       xyz="0 0 -1" />
-    <limit
-      lower="-3.14"
-      upper="3.14"
-      effort="100"
-      velocity="100" />
+    <limit lower="-0.698132" upper="0.698132" effort="1000" velocity="1.0" />
   </joint>
   <link
@@ -173,5 +171,5 @@
         xyz="7.10743075504894E-09 -3.0012958229797E-09 -0.0112499999237069"
         rpy="0 0 0" />
-      <mass
+      <!-- <mass
         value="0.0307417074716638" />
       <inertia
@@ -181,5 +179,7 @@
         iyy="5.94711068513598E-06"
         iyz="-6.03807311086712E-15"
-        izz="8.17709432093612E-06" />
+        izz="8.17709432093612E-06" /> -->
+        <mass value="0.25" />
+        <inertia ixx="0.00525" ixy="0" ixz="0" iyy="0.00035" iyz="0" izz="0.00525" />
     </inertial>
     <visual>
@@ -211,5 +211,5 @@
     type="revolute">
     <origin
-      xyz="0.639118924633511 0.284499999999994 -0.158749999999999"
+      xyz="0.639118924633511 0.284499999999994 -0.17"
       rpy="0 0 0" />
     <parent
@@ -219,9 +219,5 @@
     <axis
       xyz="0 0 -1" />
-    <limit
-      lower="-3.14"
-      upper="3.14"
-      effort="100"
-      velocity="100" />
+    <limit lower="-0.698132" upper="0.698132" effort="1000" velocity="1.0" />
   </joint>
   <link
@@ -285,5 +281,5 @@
     <inertial>
       <origin
-        xyz="-1.11022302462516E-16 -8.32667268468867E-17 0.0379999999999999"
+        xyz="-1.11022302462516E-16 -8.32667268468867E-17 -0.038"
         rpy="0 0 0" />
       <mass
@@ -393,4 +389,5 @@
       velocity="100" />
   </joint>
+<!-- /////////////////////////////// -->
   <link
     name="C16_Link">

File: src/carver_description/urdf/gazebo_control.xacro (robot description, xacro)
@@ -48,6 +48,6 @@
   <xacro:include filename="$(find carver_description)/urdf/gazebo.xacro" />
   <!-- Actuator configurations -->
-  <xacro:carver_wheel_transmission wheel_prefix="front_left_steering_front_right" />
   <xacro:carver_wheel_transmission wheel_prefix="front_left_steering_front_left" />
+  <xacro:carver_wheel_transmission wheel_prefix="front_right_steering_front_right" />
   <xacro:carver_wheel_transmission wheel_prefix="base_rear_left" />
   <xacro:carver_wheel_transmission wheel_prefix="base_rear_right" />
@@ -94,5 +94,5 @@
     <kd value="1.0"/>
   </gazebo>
-  <gazebo reference="front_right_steering_front_left_wheel_joint">
+  <gazebo reference="front_right_steering_front_right_wheel_joint">
     <mu1>10.0</mu1>
     <mu2>10.0</mu2>
