Commit message: add imu and fix urdf and add robot localization package

File: src/carver_description/urdf/carver.urdf.xacro (robot description, xacro)
@@ -7,20 +7,22 @@
   <xacro:include filename="$(find carver_description)/urdf/laser.xacro" />
   <xacro:include filename="$(find carver_description)/urdf/gps.xacro" />
-<link
+  <link
     name="base_link">
-    <inertial>
+    <!-- <inertial>
       <origin
         xyz="0.0765717108056987 -0.000305321354473288 0.182746551264274"
         rpy="0 0 0" />
-      <mass
-        value="224.620223914356" />
-      <inertia
-        ixx="11.108875181717"
-        ixy="-0.000143787949337127"
-        ixz="-0.00666553671990701"
-        iyy="35.7202876824402"
-        iyz="-0.00132350955436525"
-        izz="40.7667100665166" />
-    </inertial>
+      <mass value="2.1557" />
+      <inertia
+        ixx="0.1286"
+        ixy="0"
+        ixz="0"
+        iyy="0.3070"
+        iyz="0"
+        izz="0.4031" />
+    </inertial> -->
+    <xacro:inertial_box mass="3.0" x="0.63598" y="0.79085" z="0.10">
+        <origin xyz="0.0765717108056987 -0.000305321354473288 0.182746551264274" rpy="0 0 0"/>
+    </xacro:inertial_box>
     <visual>
       <origin
@@ -59,15 +61,12 @@
         xyz="-6.87012402522669E-09 3.51066137271872E-09 -0.0112499999237069"
         rpy="0 0 0" />
-      <!-- <mass
-        value="0.0307417074716638" />
-      <inertia
-        ixx="5.15827058483555E-06"
-        ixy="2.87694711205719E-08"
-        ixz="-2.37787643316582E-12"
-        iyy="5.94711293506547E-06"
-        iyz="1.79592218418332E-13"
-        izz="8.17709432093611E-06" /> -->
-        <mass value="0.25" />
-        <inertia ixx="0.00525" ixy="0" ixz="0" iyy="0.00035" iyz="0" izz="0.00525" />
+      <mass value="0.1" />
+      <inertia
+        ixx="0.00525"
+        ixy="0.0"
+        ixz="0.0"
+        iyy="0.00035"
+        iyz="0.0"
+        izz="0.00525" />
     </inertial>
     <visual>
@@ -99,5 +98,5 @@
     type="revolute">
     <origin
-      xyz="0.639118924633511 -0.284499999999994 -0.17"
+      xyz="0.639118924633511 -0.284499999999994 -0.158749999999999"
       rpy="0 0 0" />
     <parent
@@ -107,22 +106,21 @@
     <axis
       xyz="0 0 -1" />
-    <limit lower="-0.698132" upper="0.698132" effort="1000" velocity="1.0" />
+    <limit lower="-1.49" upper="1.49" effort="1000" velocity="1.0" />
+    <dynamics damping="1.0" friction="2.0"/>
   </joint>
   <link
     name="front_right_wheel_Link">
-    <inertial>
+    <!-- <inertial>
       <origin
         xyz="0.00138386531093282 8.32667268468867E-17 0.0379747931765428"
         rpy="0 0 0" />
-      <mass
-        value="5.024500013847" />
-      <inertia
-        ixx="0.0459745995956163"
-        ixy="8.73502726855944E-19"
-        ixz="0.00152760354434749"
-        iyy="0.0459189311540779"
-        iyz="2.21482778889901E-18"
-        izz="0.0878380602731089" />
-    </inertial>
+      <mass value="0.5" />
+      <inertia ixx="0.01055" ixy="0" ixz="0" iyy="0.00075" iyz="0" izz="0.01055" />
+    </inertial> -->
+    <xacro:inertial_cylinder mass="0.1" length="0.65" radius="0.175">
+      <origin
+        xyz="0.00138386531093282 8.32667268468867E-17 0.0379747931765428"
+        rpy="0 0 0" />
+    </xacro:inertial_cylinder>
     <visual>
       <origin
@@ -171,15 +169,12 @@
         xyz="7.10743075504894E-09 -3.0012958229797E-09 -0.0112499999237069"
         rpy="0 0 0" />
-      <!-- <mass
-        value="0.0307417074716638" />
-      <inertia
-        ixx="5.15827283476504E-06"
-        ixy="-2.88003004005144E-08"
-        ixz="2.38464111309773E-12"
-        iyy="5.94711068513598E-06"
-        iyz="-6.03807311086712E-15"
-        izz="8.17709432093612E-06" /> -->
-        <mass value="0.25" />
-        <inertia ixx="0.00525" ixy="0" ixz="0" iyy="0.00035" iyz="0" izz="0.00525" />
+      <mass value="0.1" />
+      <inertia
+        ixx="0.00525"
+        ixy="0.0"
+        ixz="0.0"
+        iyy="0.00035"
+        iyz="0.0"
+        izz="0.00525" />
     </inertial>
     <visual>
@@ -211,5 +206,5 @@
     type="revolute">
     <origin
-      xyz="0.639118924633511 0.284499999999994 -0.17"
+      xyz="0.639118924633511 0.284499999999994 -0.158749999999999"
       rpy="0 0 0" />
     <parent
@@ -219,22 +214,21 @@
     <axis
       xyz="0 0 -1" />
-    <limit lower="-0.698132" upper="0.698132" effort="1000" velocity="1.0" />
+    <limit lower="-1.49" upper="1.49" effort="1000" velocity="1.0" />
+    <dynamics damping="1.0" friction="2.0"/>
   </joint>
   <link
     name="front_left_wheel_Link">
-    <inertial>
+    <!-- <inertial>
       <origin
         xyz="0.00138386531093293 1.38777878078145E-16 -0.0379747931765427"
         rpy="0 0 0" />
-      <mass
-        value="5.02450001384701" />
-      <inertia
-        ixx="0.0459745995956163"
-        ixy="4.79764755280667E-19"
-        ixz="-0.00152760354434749"
-        iyy="0.0459189311540779"
-        iyz="-2.40802616071845E-18"
-        izz="0.0878380602731089" />
-    </inertial>
+      <mass value="0.5" />
+      <inertia ixx="0.01055" ixy="0" ixz="0" iyy="0.00075" iyz="0" izz="0.01055" />
+    </inertial> -->
+    <xacro:inertial_cylinder mass="0.1" length="0.65" radius="0.175">
+      <origin
+        xyz="0.00138386531093293 1.38777878078145E-16 -0.0379747931765427"
+        rpy="0 0 0" />
+    </xacro:inertial_cylinder>
     <visual>
       <origin
@@ -279,18 +273,16 @@
   <link
     name="rear_right_wheel_Link">
-    <inertial>
-      <origin
-        xyz="-1.11022302462516E-16 -8.32667268468867E-17 -0.038"
-        rpy="0 0 0" />
-      <mass
-        value="5.024500013847" />
-      <inertia
-        ixx="0.0459189311540779"
-        ixy="-1.56634920793041E-17"
-        ixz="1.5500519296842E-19"
-        iyy="0.045918931154078"
-        iyz="2.98988825793E-19"
-        izz="0.0878937287146473" />
-    </inertial>
+    <!-- <inertial>
+      <origin
+        xyz="-1.11022302462516E-16 -8.32667268468867E-17 0.0379999999999999"
+        rpy="0 0 0" />
+      <mass value="0.5" />
+      <inertia ixx="0.01055" ixy="0" ixz="0" iyy="0.00075" iyz="0" izz="0.01055" />
+    </inertial> -->
+    <xacro:inertial_cylinder mass="0.1" length="0.65" radius="0.175">
+      <origin
+        xyz="-1.11022302462516E-16 -8.32667268468867E-17 0.0379999999999999"
+        rpy="0 0 0" />
+    </xacro:inertial_cylinder>
     <visual>
       <origin
@@ -335,18 +327,16 @@
   <link
     name="rear_left_wheel_Link">
-    <inertial>
+    <!-- <inertial>
       <origin
         xyz="-1.11022302462516E-16 -5.55111512312578E-17 -0.038"
         rpy="0 0 0" />
-      <mass
-        value="5.024500013847" />
-      <inertia
-        ixx="0.0459189311540779"
-        ixy="-1.69253786030664E-17"
-        ixz="-3.82127958527989E-20"
-        iyy="0.0459189311540779"
-        iyz="-3.5370156940672E-19"
-        izz="0.0878937287146472" />
-    </inertial>
+      <mass value="0.5" />
+      <inertia ixx="0.01055" ixy="0" ixz="0" iyy="0.00075" iyz="0" izz="0.01055" />
+    </inertial> -->
+    <xacro:inertial_cylinder mass="0.1" length="0.65" radius="0.175">
+      <origin
+        xyz="-1.11022302462516E-16 -5.55111512312578E-17 0.0379999999999999"
+        rpy="0 0 0" />
+    </xacro:inertial_cylinder>
     <visual>
       <origin
@@ -394,14 +384,14 @@
     <inertial>
       <origin
-        xyz="-0.00088474978448877 1.07190642272392E-07 0.00143612694647577"
+        xyz="-0.00088474978448877 0.0 0.00143612694647577"
         rpy="0 0 0" />
       <mass
-        value="0.663324628749119" />
+        value="0.01" />
       <inertia
         ixx="0.000791421263365419"
-        ixy="1.38226469561758E-09"
-        ixz="-5.15681751766988E-06"
+        ixy="0.0"
+        ixz="0.0"
         iyy="0.000800507843146539"
-        iyz="1.51968163395454E-09"
+        iyz="0.00"
         izz="0.000866550903215115" />
     </inertial>
@@ -450,5 +440,5 @@
         rpy="0 0 0" />
       <mass
-        value="0.015352262982903" />
+        value="0.01" />
       <inertia
         ixx="1.39361946583924E-05"
@@ -496,4 +486,41 @@
       xyz="0 0 0" />
   </joint>
+  <!-- <gazebo reference="T265_Link">
+      <material>Gazebo/Yellow</material>
+      <sensor name="sensor_camera" type="depth">
+          <pose>0.0 0.0 0.0 0.0 0.0 0.0</pose>
+          <always_on>1</always_on>
+          <update_rate>10</update_rate>
+          <visualize>1</visualize>
+          <camera name="carver_camera">
+          <image>
+              <format>R8G8B8</format>
+              <width>400</width>
+              <height>400</height>
+          </image>
+          <clip>
+              <near>0.01</near>
+              <far>10.0</far>
+          </clip>
+          </camera>
+          <plugin name="gazebo_ros_depth_camera_sensor" filename="libgazebo_ros_camera.so">
+              <ros>
+                  <namespace>/carver</namespace>
+                  <ros-args>
+                      <remap from="carver_camera/image_raw" to="carver_camera/image"/>
+                      <remap from="carver_camera/image_depth" to="carver_camera/depth/camera_image_depth"/>
+                      <remap from="carver_camera/camera_info" to="carver_camera/camera_info_raw"/>
+                      <remap from="carver_camera/camera_info_depth" to="carver_camera/camera_info_depth"/>
+                      <remap from="carver_camera/points" to="carver_camera/camera_points"/>
+                  </ros-args>
+              </ros>
+              <camera_name>T265</camera_name>
+              <frame_name>T265_Link</frame_name>
+              <hack_baseline>0.07</hack_baseline>
+              <min_depth>0.001</min_depth>
+          </plugin>
+      </sensor>
+  </gazebo>
+   -->
   <link
     name="L515_Link">
@@ -503,5 +530,5 @@
         rpy="0 0 0" />
       <mass
-        value="0.0519003008833496" />
+        value="0.01" />
       <inertia
         ixx="2.29233885806633E-05"
@@ -556,5 +583,5 @@
         rpy="0 0 0" />
       <mass
-        value="0.911976961838322" />
+        value="0.01" />
       <inertia
         ixx="0.00155787250018401"

File: src/carver_description/urdf/gazebo.xacro (robot description, xacro)
@@ -6,5 +6,4 @@
             <actuator name="${wheel_prefix}_wheel_motor">
                 <hardwareInterface>hardware_interface/VelocityJointInterface</hardwareInterface>
-                <mechanicalReduction>1</mechanicalReduction>
             </actuator>
             <joint name="${wheel_prefix}_wheel_joint">
@@ -18,5 +17,4 @@
             <actuator name="${wheel_prefix}_sterring_motor">
                 <hardwareInterface>hardware_interface/EffortJointInterface</hardwareInterface>
-                <mechanicalReduction>1</mechanicalReduction>
             </actuator>
             <joint name="${wheel_prefix}_sterring_joint">

File: src/carver_description/urdf/gazebo_control.xacro (robot description, xacro)
@@ -5,5 +5,5 @@
     <plugin filename="libgazebo_ros2_control.so" name="gazebo_ros2_control">
       <!-- Path to your ROS2 control config -->
-      <parameters>$(find carver_gazebo)/config/controllers.yaml</parameters>
+      <parameters>$(find carver_description)/config/controllers.yaml</parameters>
     </plugin>
   </gazebo>
@@ -15,33 +15,51 @@
     <!-- Four wheel joints, using velocity commands -->
     <joint name="front_left_steering_front_left_wheel_joint">
-      <state_interface name="position"/>
+      <state_interface name="position">
+        <param name="initial_value">0.0</param>
+      </state_interface>
       <state_interface name="velocity"/>
+      <state_interface name="effort"/>
     </joint>
     <joint name="front_right_steering_front_right_wheel_joint">
-      <state_interface name="position"/>
+      <state_interface name="position">
+        <param name="initial_value">0.0</param>
+      </state_interface>
       <state_interface name="velocity"/>
+      <state_interface name="effort"/>
     </joint>
     <joint name="base_rear_left_wheel_joint">
       <command_interface name="velocity"/>
-      <state_interface name="position"/>
+      <state_interface name="position">
+        <param name="initial_value">0.0</param>
+      </state_interface>
       <state_interface name="velocity"/>
+      <state_interface name="effort"/>
     </joint>
     <joint name="base_rear_right_wheel_joint">
       <command_interface name="velocity"/>
-      <state_interface name="position"/>
+      <state_interface name="position">
+        <param name="initial_value">0.0</param>
+      </state_interface>
       <state_interface name="velocity"/>
+      <state_interface name="effort"/>
     </joint>
     <!-- Steering joints, using a position interface -->
     <joint name="base_front_left_sterring_joint">
-      <command_interface name="position"/>
-      <state_interface name="position">
-      </state_interface>
+      <command_interface name="position">
+      </command_interface>
+        <state_interface name="position">
+          <param name="initial_value">0.0</param>
+        </state_interface>
       <state_interface name="velocity"/>
+      <state_interface name="effort"/>
     </joint>
     <joint name="base_front_right_sterring_joint">
-      <command_interface name="position"/>
-      <state_interface name="position">
-      </state_interface>
+      <command_interface name="position">
+      </command_interface>
+        <state_interface name="position">
+          <param name="initial_value">0.0</param>
+        </state_interface>
       <state_interface name="velocity"/>
+      <state_interface name="effort"/>
     </joint>
   </ros2_control>
@@ -59,5 +77,5 @@
   <!-- <xacro:gazebo_gps link_name="GPS_Link" topic="/gps/fix" frame_name="GPS_Link" /> -->
   <!-- Gazebo friction/contact parameters -->
-  <gazebo>
+  <!-- <gazebo>
     <mu1 value="10"/>
     <mu2 value="10"/>
@@ -67,5 +85,5 @@
     <minDepth value="0.001"/>
     <maxContacts value="64"/>
-  </gazebo>
+  </gazebo> -->
   <gazebo reference="base_link">
     <minDepth>0.0001</minDepth>
@@ -73,5 +91,5 @@
     <kd value="1.0"/>
   </gazebo>
-  <gazebo reference="front_left_sterring_Link">
+  <!-- <gazebo reference="front_left_sterring_Link">
     <mu1>10.0</mu1>
     <mu2>10.0</mu2>
@@ -86,6 +104,6 @@
     <kp value="1000000.0"/>
     <kd value="1.0"/>
-  </gazebo>
-  <!-- <gazebo reference="front_left_steering_front_left_wheel_joint">
+  </gazebo> -->
+  <gazebo reference="front_left_wheel_Link">
     <mu1>10.0</mu1>
     <mu2>10.0</mu2>
@@ -94,5 +112,5 @@
     <kd value="1.0"/>
   </gazebo>
-  <gazebo reference="front_right_steering_front_right_wheel_joint">
+  <gazebo reference="front_right_wheel_Link">
     <mu1>10.0</mu1>
     <mu2>10.0</mu2>
@@ -100,5 +118,5 @@
     <kp value="1000000.0"/>
     <kd value="1.0"/>
-  </gazebo> -->
+  </gazebo>
   <gazebo reference="rear_left_wheel_Link">
     <mu1>10.0</mu1>

File: src/carver_description/urdf/gps.xacro (robot description, xacro)
@@ -8,5 +8,5 @@
         rpy="0 0 0" />
       <mass
-        value="0.157649586184773" />
+        value="0.01" />
       <inertia
         ixx="0.000226882899026971"
@@ -54,3 +54,23 @@
       xyz="0 0 0" />
   </joint>
+<gazebo reference="GPS_Link">
+  <sensor name="gps_sensor" type="gps">
+    <always_on>true</always_on>
+    <update_rate>30</update_rate>
+    <gps>
+      <noise>
+        <type>gaussian</type>
+        <mean>0.0</mean>
+        <stddev>0.1</stddev>
+      </noise>
+    </gps>
+    <plugin name="gps_plugin" filename="libgazebo_ros_gps_sensor.so">
+      <ros>
+        <namespace>/gps</namespace>
+        <remapping>~/out:=data</remapping>
+      </ros>
+      <frame_name>GPS_Link</frame_name>
+    </plugin>
+  </sensor>
+</gazebo>
 </robot>

File: src/carver_description/urdf/imu.xacro (robot description, xacro)
@@ -8,14 +8,12 @@
         rpy="0 0 0" />
       <mass
-        value="0.000983130183652042" />
+        value="0.01" />
       <inertia
-        ixx="2.7278081479223E-08"
-        ixy="-1.86463715352951E-11"
-        ixz="-1.83135757569472E-11"
-        iyy="4.80453464098755E-08"
-        iyz="1.81575171892503E-12"
-        izz="7.48563776021962E-08" />
+        ixx="1e-7" ixy="0" ixz="0"
+        iyy="1e-7" iyz="0"
+        izz="1e-7"
+      />
     </inertial>
-    <visual>
+    <visual name='IMU_R_Link_visual'>
       <origin
         xyz="0 0 0"
@@ -25,8 +23,10 @@
           filename="file://$(find carver_description)/meshes/IMU_R_Link.dae" />
       </geometry>
-      <material
-        name="">
-        <color
-          rgba="0.792156862745098 0.819607843137255 0.933333333333333 1" />
+      <material name='imu_r_material'>
+        <color rgba="0.75 0.75 0.75 1" />
+          <ambient>0.1 0.1 0.1 1</ambient>
+          <diffuse>0.1 0.1 0.2 1</diffuse>
+          <specular>0 0 0 0</specular>
+          <emissive>0 0 0 1</emissive>
       </material>
     </visual>
@@ -61,14 +61,12 @@
         rpy="0 0 0" />
       <mass
-        value="0.000983130183652038" />
+        value="0.01" />
       <inertia
-        ixx="2.7278081479223E-08"
-        ixy="-1.86463715354835E-11"
-        ixz="-1.83135757570018E-11"
-        iyy="4.80453464098757E-08"
-        iyz="1.8157517189233E-12"
-        izz="7.48563776021965E-08" />
+        ixx="1e-7" ixy="0" ixz="0"
+        iyy="1e-7" iyz="0"
+        izz="1e-7"
+      />
     </inertial>
-    <visual>
+    <visual name='IMU_L_Link_visual'>
       <origin
         xyz="0 0 0"
@@ -78,8 +76,10 @@
           filename="file://$(find carver_description)/meshes/IMU_L_Link.dae" />
       </geometry>
-      <material
-        name="">
-        <color
-          rgba="0.792156862745098 0.819607843137255 0.933333333333333 1" />
+      <material name='imu_l_material'>
+        <color rgba="0.75 0.75 0.75 1" />
+          <ambient>0.1 0.1 0.1 1</ambient>
+          <diffuse>0.1 0.1 0.2 1</diffuse>
+          <specular>0 0 0 0</specular>
+          <emissive>0 0 0 1</emissive>
       </material>
     </visual>
@@ -107,3 +107,157 @@
       xyz="0 0 0" />
   </joint>
+  <gazebo reference="IMU_R_Link">
+      <gravity>true</gravity>
+      <sensor name="IMU_R" type="imu">
+      <always_on>true</always_on>
+      <update_rate>100</update_rate>
+      <visualize>true</visualize>
+      <imu>
+          <orientation>
+          <x>
+              <noise type="gaussian">
+              <mean>0.0</mean>
+              <stddev>2e-3</stddev>
+              </noise>
+          </x>
+          <y>
+              <noise type="gaussian">
+              <mean>0.0</mean>
+              <stddev>2e-3</stddev>
+              </noise>
+          </y>
+          <z>
+              <noise type="gaussian">
+              <mean>0.0</mean>
+              <stddev>2e-3</stddev>
+              </noise>
+          </z>
+          </orientation>
+          <angular_velocity>
+          <x>
+              <noise type="gaussian">
+              <mean>0.0</mean>
+              <stddev>2e-4</stddev>
+              </noise>
+          </x>
+          <y>
+              <noise type="gaussian">
+              <mean>0.0</mean>
+              <stddev>2e-4</stddev>
+              </noise>
+          </y>
+          <z>
+              <noise type="gaussian">
+              <mean>0.0</mean>
+              <stddev>2e-4</stddev>
+              </noise>
+          </z>
+          </angular_velocity>
+          <linear_acceleration>
+          <x>
+              <noise type="gaussian">
+              <mean>0.0</mean>
+              <stddev>1.7e-2</stddev>
+              </noise>
+          </x>
+          <y>
+              <noise type="gaussian">
+              <mean>0.0</mean>
+              <stddev>1.7e-2</stddev>
+              </noise>
+          </y>
+          <z>
+              <noise type="gaussian">
+              <mean>0.0</mean>
+              <stddev>1.7e-2</stddev>
+              </noise>
+          </z>
+          </linear_acceleration>
+      </imu>
+      <plugin name="IMU_R" filename="libgazebo_ros_imu_sensor.so">
+          <initial_orientation_as_reference>false</initial_orientation_as_reference>
+          <frame_name>IMU_R_Link</frame_name>
+          <ros>
+          <remapping>~/out:=imu_R</remapping>
+          </ros>
+      </plugin>
+      </sensor>
+  </gazebo>
+  <gazebo reference="IMU_L_Link">
+      <gravity>true</gravity>
+      <sensor name="IMU_L" type="imu">
+      <always_on>true</always_on>
+      <update_rate>100</update_rate>
+      <visualize>true</visualize>
+      <imu>
+          <orientation>
+          <x>
+              <noise type="gaussian">
+              <mean>0.0</mean>
+              <stddev>2e-3</stddev>
+              </noise>
+          </x>
+          <y>
+              <noise type="gaussian">
+              <mean>0.0</mean>
+              <stddev>2e-3</stddev>
+              </noise>
+          </y>
+          <z>
+              <noise type="gaussian">
+              <mean>0.0</mean>
+              <stddev>2e-3</stddev>
+              </noise>
+          </z>
+          </orientation>
+          <angular_velocity>
+          <x>
+              <noise type="gaussian">
+              <mean>0.0</mean>
+              <stddev>2e-4</stddev>
+              </noise>
+          </x>
+          <y>
+              <noise type="gaussian">
+              <mean>0.0</mean>
+              <stddev>2e-4</stddev>
+              </noise>
+          </y>
+          <z>
+              <noise type="gaussian">
+              <mean>0.0</mean>
+              <stddev>2e-4</stddev>
+              </noise>
+          </z>
+          </angular_velocity>
+          <linear_acceleration>
+          <x>
+              <noise type="gaussian">
+              <mean>0.0</mean>
+              <stddev>1.7e-2</stddev>
+              </noise>
+          </x>
+          <y>
+              <noise type="gaussian">
+              <mean>0.0</mean>
+              <stddev>1.7e-2</stddev>
+              </noise>
+          </y>
+          <z>
+              <noise type="gaussian">
+              <mean>0.0</mean>
+              <stddev>1.7e-2</stddev>
+              </noise>
+          </z>
+          </linear_acceleration>
+      </imu>
+      <plugin name="IMU_L" filename="libgazebo_ros_imu_sensor.so">
+          <initial_orientation_as_reference>false</initial_orientation_as_reference>
+          <frame_name>IMU_L_Link</frame_name>
+          <ros>
+          <remapping>~/out:=imu_L</remapping>
+          </ros>
+      </plugin>
+      </sensor>
+  </gazebo>
 </robot>
