Commit message: add imu and fix urdf and add robot localization package

File: src/carver_description/urdf/inertial_macros.xacro (robot description, xacro)
@@ -1,31 +1,40 @@
 <?xml version="1.0"?>
-<robot xmlns:xacro="http://ros.org/wiki/xacro">
-    <xacro:macro name="sphere_inertial_matrix" params="m r">
+<robot xmlns:xacro="http://www.ros.org/wiki/xacro" >
+    <!-- Specify some standard inertial calculations https://en.wikipedia.org/wiki/List_of_moments_of_inertia -->
+    <!-- These make use of xacro's mathematical functionality -->
+    <xacro:macro name="inertial_sphere" params="mass radius *origin">
         <inertial>
-            <origin xyz="0.0 0.0 0.0" />
-            <mass value="${m}" />
-            <inertia ixx="${2*m*r*r/5}" ixy="0" ixz="0"
-                     iyy="${2*m*r*r/5}" iyz="0"
-                     izz="${2*m*r*r/5}" />
+            <xacro:insert_block name="origin"/>
+            <mass value="${mass}" />
+            <inertia ixx="${(2/5) * mass * (radius*radius)}" ixy="0.0" ixz="0.0"
+                    iyy="${(2/5) * mass * (radius*radius)}" iyz="0.0"
+                    izz="${(2/5) * mass * (radius*radius)}" />
         </inertial>
     </xacro:macro>
-    <!-- Zylinder -->
-    <xacro:macro name="cylinder_inertial_matrix" params="m r h d">
+    <xacro:macro name="inertial_box" params="mass x y z *origin">
         <inertial>
-            <origin xyz="0 0 ${d}" />
-            <mass value="${m}" />
-            <inertia ixx="${(1/12) * m * (3*r*r + h*h) + m*d*d}" ixy="0" ixz="0"
-                    iyy="${(1/12) * m * (3*r*r + h*h)}" iyz="0"
-                    izz="${(1/2) * m * r*r}" />
+            <xacro:insert_block name="origin"/>
+            <mass value="${mass}" />
+            <inertia ixx="${(1/12) * mass * (y*y+z*z)}" ixy="0.0" ixz="0.0"
+                    iyy="${(1/12) * mass * (x*x+z*z)}" iyz="0.0"
+                    izz="${(1/12) * mass * (x*x+y*y)}" />
         </inertial>
     </xacro:macro>
-    <!-- Quader -->
-    <xacro:macro name="box_inertial_matrix" params="m w l h">
+    <xacro:macro name="inertial_cylinder" params="mass length radius *origin">
         <inertial>
-            <origin xyz="0.0 0.0 0.0" />
-            <mass value="${m}" />
-            <inertia ixx="${m*(w*w+h*h)/12}" ixy = "0" ixz = "0"
-                     iyy="${m*(h*h+l*l)/12}" iyz = "0"
-                     izz="${m*(w*w+l*l)/12}" />
+            <xacro:insert_block name="origin"/>
+            <mass value="${mass}" />
+            <inertia ixx="${(1/12) * mass * (3*radius*radius + length*length)}" ixy="0.0" ixz="0.0"
+                    iyy="${(1/12) * mass * (3*radius*radius + length*length)}" iyz="0.0"
+                    izz="${(1/2) * mass * (radius*radius)}" />
+        </inertial>
+    </xacro:macro>
+    <xacro:macro name="inertial_flip_cylinder" params="mass length radius *origin">
+        <inertial>
+            <xacro:insert_block name="origin"/>
+            <mass value="${mass}" />
+            <inertia ixx="${(1/12) * mass * (3*radius*radius + length*length)}" ixy="0.0" ixz="0.0"
+                    iyy="${(1/2) * mass * (radius*radius)}" iyz="0.0"
+                    izz="${(1/12) * mass * (3*radius*radius + length*length)}" />
         </inertial>
     </xacro:macro>

File: src/carver_description/urdf/laser.xacro (robot description, xacro)
@@ -16,5 +16,5 @@
         rpy="0 0 0" />
       <mass
-        value="0.0328083847884842" />
+        value="0.01" />
       <inertia
         ixx="1.08465576772131E-05"
@@ -71,5 +71,5 @@
         rpy="0 0 0" />
       <mass
-        value="0.0328083843446528" />
+        value="0.01" />
       <inertia
         ixx="1.0846557670466E-05"
