Commit message: add robot ekf

File: src/carver_description/urdf/imu.xacro (robot description, xacro)
@@ -108,4 +108,5 @@
   </joint>
   <gazebo reference="IMU_R_Link">
+      <material>Gazebo/Yellow</material>
       <gravity>true</gravity>
       <sensor name="IMU_R" type="imu">
@@ -185,4 +186,5 @@
   </gazebo>
   <gazebo reference="IMU_L_Link">
+      <material>Gazebo/Yellow</material>
       <gravity>true</gravity>
       <sensor name="IMU_L" type="imu">
