Commit message: remove marge lidar

File: src/carver_description/urdf/gazebo.xacro (robot description, xacro)
@@ -1,4 +1,4 @@
 <?xml version="1.0"?>
-<robot name="carver_description" xmlns:xacro="http://ros.org/wiki/xacro">
+<robot xmlns:xacro="http://ros.org/wiki/xacro">
   <xacro:macro name="carver_wheel_transmission" params="wheel_prefix">
         <transmission name="${wheel_prefix}_wheel_trans" type="SimpleTransmission">
@@ -23,140 +23,3 @@
         </transmission>
   </xacro:macro>
-    <xacro:macro name="gazebo_laser" params="frame_prefix">
-        <gazebo reference="${frame_prefix}_link">
-            <sensor name="laser" type="ray">
-            <always_on>true</always_on>
-            <visualize>false</visualize>
-            <update_rate>10</update_rate>
-            <ray>
-                <scan>
-                <horizontal>
-                    <samples>120</samples>
-                    <resolution>1.000000</resolution>
-                    <min_angle>-3.14159</min_angle>
-                    <max_angle>3.14159</max_angle>
-                </horizontal>
-                </scan>
-                <range>
-                <min>0.3</min>
-                <max>15.0</max>
-                <resolution>0.015</resolution>
-                </range>
-                <noise>
-                <type>gaussian</type>
-                <mean>0.0</mean>
-                <stddev>0.01</stddev>
-                </noise>
-            </ray>
-            <plugin name="scan" filename="libgazebo_ros_ray_sensor.so">
-                <ros>
-                <remapping>~/out:=scan</remapping>
-                </ros>
-                <output_type>sensor_msgs/LaserScan</output_type>
-                <frame_name>laser</frame_name>
-            </plugin>
-            </sensor>
-        </gazebo>
-    </xacro:macro>
-    <xacro:macro name="gazebo_imu" params="link_name topic frame_name">
-    <gazebo reference="${link_name}">
-        <gravity>true</gravity>
-        <sensor name="${link_name}_imu" type="imu">
-        <always_on>true</always_on>
-        <update_rate>100</update_rate>
-        <visualize>true</visualize>
-        <imu>
-            <orientation>
-            <x>
-                <noise type="gaussian">
-                <mean>0.0</mean>
-                <stddev>2e-3</stddev>
-                </noise>
-            </x>
-            <y>
-                <noise type="gaussian">
-                <mean>0.0</mean>
-                <stddev>2e-3</stddev>
-                </noise>
-            </y>
-            <z>
-                <noise type="gaussian">
-                <mean>0.0</mean>
-                <stddev>2e-3</stddev>
-                </noise>
-            </z>
-            </orientation>
-            <angular_velocity>
-            <x>
-                <noise type="gaussian">
-                <mean>0.0</mean>
-                <stddev>2e-4</stddev>
-                </noise>
-            </x>
-            <y>
-                <noise type="gaussian">
-                <mean>0.0</mean>
-                <stddev>2e-4</stddev>
-                </noise>
-            </y>
-            <z>
-                <noise type="gaussian">
-                <mean>0.0</mean>
-                <stddev>2e-4</stddev>
-                </noise>
-            </z>
-            </angular_velocity>
-            <linear_acceleration>
-            <x>
-                <noise type="gaussian">
-                <mean>0.0</mean>
-                <stddev>1.7e-2</stddev>
-                </noise>
-            </x>
-            <y>
-                <noise type="gaussian">
-                <mean>0.0</mean>
-                <stddev>1.7e-2</stddev>
-                </noise>
-            </y>
-            <z>
-                <noise type="gaussian">
-                <mean>0.0</mean>
-                <stddev>1.7e-2</stddev>
-                </noise>
-            </z>
-            </linear_acceleration>
-        </imu>
-        <plugin name="two_wheeled_robot_imu" filename="libgazebo_ros_imu_sensor.so">
-            <initial_orientation_as_reference>false</initial_orientation_as_reference>
-            <frame_name>${frame_name}_imu_link</frame_name>
-            <ros>
-            <remapping>~/out:=${topic}/imu</remapping>
-            </ros>
-        </plugin>
-        </sensor>
-    </gazebo>
-    </xacro:macro>
-    <xacro:macro name="gazebo_gps" params="link_name topic frame_name">
-    <gazebo reference="${link_name}">
-        <gravity>true</gravity>
-        <sensor name="${link_name}_gps" type="gps">
-        <always_on>true</always_on>
-        <update_rate>5</update_rate>
-        <visualize>true</visualize>
-        <pose>0 0 0 0 0 0</pose>
-        <gps>
-            <!-- Adjust smoothing or add noise parameters as required -->
-            <position_smoothing>0.5</position_smoothing>
-        </gps>
-        <plugin name="gazebo_ros_gps_sensor" filename="libgazebo_ros_gps_plugin.so">
-            <ros>
-            <remapping>~/out:=${topic}</remapping>
-            </ros>
-            <topicName>${topic}</topicName>
-            <frameName>${frame_name}</frameName>
-        </plugin>
-        </sensor>
-    </gazebo>
-    </xacro:macro>
 </robot>

File: src/carver_description/urdf/gazebo_control.xacro (robot description, xacro)
@@ -83,8 +83,4 @@
   <xacro:carver_steering_hinge_transmission wheel_prefix="base_front_right" />
   <xacro:carver_steering_hinge_transmission wheel_prefix="base_front_left" />
-  <!-- <xacro:gazebo_laser frame_prefix="laser" /> -->
-  <!-- <xacro:gazebo_imu link_name="IMU_R_Link" topic="/imu_right" frame_name="IMU_R_Link" />
-  <xacro:gazebo_imu link_name="IMU_L_Link" topic="/imu_left" frame_name="IMU_L_Link" /> -->
-  <!-- <xacro:gazebo_gps link_name="GPS_Link" topic="/gps/fix" frame_name="GPS_Link" /> -->
   <!-- Gazebo friction/contact parameters -->
   <!-- <gazebo>

File: src/carver_description/urdf/laser.xacro (robot description, xacro)
@@ -147,5 +147,5 @@
             <plugin name="scan_LB" filename="libgazebo_ros_ray_sensor.so">
                 <ros>
-                <remapping>~/out:=scan_LB</remapping>
+                <remapping>~/out:=lidar_2/scan</remapping>
                 </ros>
                 <output_type>sensor_msgs/LaserScan</output_type>
@@ -182,5 +182,5 @@
             <plugin name="scan_RF" filename="libgazebo_ros_ray_sensor.so">
                 <ros>
-                <remapping>~/out:=scan_RF</remapping>
+                <remapping>~/out:=lidar_1/scan</remapping>
                 </ros>
                 <output_type>sensor_msgs/LaserScan</output_type>
