Commit message: update work simple slam

File: src/carver_description/urdf/carver.xacro (robot description, xacro)
@@ -1,25 +1,13 @@
 <?xml version="1.0" encoding="utf-8"?>
 <robot name="carver_description" xmlns:xacro="http://www.ros.org/wiki/xacro">
-  <xacro:arg name="robot_namespace" default="/" />
-  <xacro:include filename="$(find carver_description)/urdf/gazebo_control.xacro" />
-  <xacro:include filename="$(find carver_description)/urdf/inertial_macros.xacro" />
-  <xacro:include filename="$(find carver_description)/urdf/imu.xacro" />
-  <xacro:include filename="$(find carver_description)/urdf/laser.xacro" />
-  <xacro:include filename="$(find carver_description)/urdf/gps.xacro" />
+  <xacro:include filename="inertial_macros.xacro" />
+  <link name="base_footprint"></link>
+  <joint name="base_joint" type="fixed">
+    <parent link="base_footprint"/>
+    <child link="base_link"/>
+    <origin xyz="0.0 0.0 0.345" rpy="0 0 0"/>
+  </joint>
   <link
     name="base_link">
-    <!-- <inertial>
-      <origin
-        xyz="0.0765717108056987 -0.000305321354473288 0.182746551264274"
-        rpy="0 0 0" />
-      <mass value="2.1557" />
-      <inertia
-        ixx="0.1286"
-        ixy="0"
-        ixz="0"
-        iyy="0.3070"
-        iyz="0"
-        izz="0.4031" />
-    </inertial> -->
     <xacro:inertial_box mass="3.0" x="0.63598" y="0.79085" z="0.10">
         <origin xyz="0.0765717108056987 -0.000305321354473288 0.182746551264274" rpy="0 0 0"/>
@@ -31,28 +19,22 @@
       <geometry>
         <mesh
-          filename="file://$(find carver_description)/meshes/base_link.STL" />
-      </geometry>
-      <material
-        name="">
-        <color
-          rgba="0.792156862745098 0.819607843137255 0.933333333333333 1" />
-      </material>
-    </visual>
-    <collision>
-      <origin
-        xyz="0 0 0"
-        rpy="0 0 0" />
-      <geometry>
-        <mesh
-          filename="file://$(find carver_description)/meshes/base_link.STL" />
-      </geometry>
-    </collision>
-  </link>
-  <link name="base_footprint"></link>
-  <joint name="world_base_joint" type="fixed">
-    <parent link="base_footprint" />
-    <child link="base_link" />
-    <origin xyz="0 0 0.345" rpy="0 0 0" />
-  </joint>
+          filename="file:///$(find carver_description)/meshes/base_link.dae" />
+      </geometry>
+      <material
+        name="">
+        <color
+          rgba="0.792156862745098 0.819607843137255 0.933333333333333 1" />
+      </material>
+    </visual>
+    <collision>
+      <origin
+        xyz="0 0 0"
+        rpy="0 0 0" />
+      <geometry>
+        <mesh
+          filename="file:///$(find carver_description)/meshes/base_link.dae" />
+      </geometry>
+    </collision>
+  </link>
   <link
     name="front_right_sterring_Link">
@@ -76,19 +58,19 @@
       <geometry>
         <mesh
-          filename="file://$(find carver_description)/meshes/front_right_sterring_Link.STL" />
-      </geometry>
-      <material
-        name="">
-        <color
-          rgba="0.792156862745098 0.819607843137255 0.933333333333333 1" />
-      </material>
-    </visual>
-    <collision>
-      <origin
-        xyz="0 0 0"
-        rpy="0 0 0" />
-      <geometry>
-        <mesh
-          filename="file://$(find carver_description)/meshes/front_right_sterring_Link.STL" />
+          filename="file:///$(find carver_description)/meshes/front_right_sterring_Link.dae" />
+      </geometry>
+      <material
+        name="">
+        <color
+          rgba="0.792156862745098 0.819607843137255 0.933333333333333 1" />
+      </material>
+    </visual>
+    <collision>
+      <origin
+        xyz="0 0 0"
+        rpy="0 0 0" />
+      <geometry>
+        <mesh
+          filename="file:///$(find carver_description)/meshes/front_right_sterring_Link.dae" />
       </geometry>
     </collision>
@@ -129,19 +111,19 @@
       <geometry>
         <mesh
-          filename="file://$(find carver_description)/meshes/front_right_wheel_Link.STL" />
-      </geometry>
-      <material
-        name="">
-        <color
-          rgba="0.792156862745098 0.819607843137255 0.933333333333333 1" />
-      </material>
-    </visual>
-    <collision>
-      <origin
-        xyz="0 0 0"
-        rpy="0 0 0" />
-      <geometry>
-        <mesh
-          filename="file://$(find carver_description)/meshes/front_right_wheel_Link.STL" />
+          filename="file:///$(find carver_description)/meshes/front_right_wheel_Link.dae" />
+      </geometry>
+      <material
+        name="">
+        <color
+          rgba="0.792156862745098 0.819607843137255 0.933333333333333 1" />
+      </material>
+    </visual>
+    <collision>
+      <origin
+        xyz="0 0 0"
+        rpy="0 0 0" />
+      <geometry>
+        <mesh
+          filename="file:///$(find carver_description)/meshes/front_right_wheel_Link.dae" />
       </geometry>
     </collision>
@@ -184,19 +166,19 @@
       <geometry>
         <mesh
-          filename="file://$(find carver_description)/meshes/front_left_sterring_Link.STL" />
-      </geometry>
-      <material
-        name="">
-        <color
-          rgba="0.792156862745098 0.819607843137255 0.933333333333333 1" />
-      </material>
-    </visual>
-    <collision>
-      <origin
-        xyz="0 0 0"
-        rpy="0 0 0" />
-      <geometry>
-        <mesh
-          filename="file://$(find carver_description)/meshes/front_left_sterring_Link.STL" />
+          filename="file:///$(find carver_description)/meshes/front_left_sterring_Link.dae" />
+      </geometry>
+      <material
+        name="">
+        <color
+          rgba="0.792156862745098 0.819607843137255 0.933333333333333 1" />
+      </material>
+    </visual>
+    <collision>
+      <origin
+        xyz="0 0 0"
+        rpy="0 0 0" />
+      <geometry>
+        <mesh
+          filename="file:///$(find carver_description)/meshes/front_left_sterring_Link.dae" />
       </geometry>
     </collision>
@@ -237,19 +219,19 @@
       <geometry>
         <mesh
-          filename="file://$(find carver_description)/meshes/front_left_wheel_Link.STL" />
-      </geometry>
-      <material
-        name="">
-        <color
-          rgba="0.792156862745098 0.819607843137255 0.933333333333333 1" />
-      </material>
-    </visual>
-    <collision>
-      <origin
-        xyz="0 0 0"
-        rpy="0 0 0" />
-      <geometry>
-        <mesh
-          filename="file://$(find carver_description)/meshes/front_left_wheel_Link.STL" />
+          filename="file:///$(find carver_description)/meshes/front_left_wheel_Link.dae" />
+      </geometry>
+      <material
+        name="">
+        <color
+          rgba="0.792156862745098 0.819607843137255 0.933333333333333 1" />
+      </material>
+    </visual>
+    <collision>
+      <origin
+        xyz="0 0 0"
+        rpy="0 0 0" />
+      <geometry>
+        <mesh
+          filename="file:///$(find carver_description)/meshes/front_left_wheel_Link.dae" />
       </geometry>
     </collision>
@@ -291,19 +273,19 @@
       <geometry>
         <mesh
-          filename="file://$(find carver_description)/meshes/rear_right_wheel_Link.STL" />
-      </geometry>
-      <material
-        name="">
-        <color
-          rgba="0.792156862745098 0.819607843137255 0.933333333333333 1" />
-      </material>
-    </visual>
-    <collision>
-      <origin
-        xyz="0 0 0"
-        rpy="0 0 0" />
-      <geometry>
-        <mesh
-          filename="file://$(find carver_description)/meshes/rear_right_wheel_Link.STL" />
+          filename="file:///$(find carver_description)/meshes/rear_right_wheel_Link.dae" />
+      </geometry>
+      <material
+        name="">
+        <color
+          rgba="0.792156862745098 0.819607843137255 0.933333333333333 1" />
+      </material>
+    </visual>
+    <collision>
+      <origin
+        xyz="0 0 0"
+        rpy="0 0 0" />
+      <geometry>
+        <mesh
+          filename="file:///$(find carver_description)/meshes/rear_right_wheel_Link.dae" />
       </geometry>
     </collision>
@@ -345,19 +327,19 @@
       <geometry>
         <mesh
-          filename="file://$(find carver_description)/meshes/rear_left_wheel_Link.STL" />
-      </geometry>
-      <material
-        name="">
-        <color
-          rgba="0.792156862745098 0.819607843137255 0.933333333333333 1" />
-      </material>
-    </visual>
-    <collision>
-      <origin
-        xyz="0 0 0"
-        rpy="0 0 0" />
-      <geometry>
-        <mesh
-          filename="file://$(find carver_description)/meshes/rear_left_wheel_Link.STL" />
+          filename="file:///$(find carver_description)/meshes/rear_left_wheel_Link.dae" />
+      </geometry>
+      <material
+        name="">
+        <color
+          rgba="0.792156862745098 0.819607843137255 0.933333333333333 1" />
+      </material>
+    </visual>
+    <collision>
+      <origin
+        xyz="0 0 0"
+        rpy="0 0 0" />
+      <geometry>
+        <mesh
+          filename="file:///$(find carver_description)/meshes/rear_left_wheel_Link.dae" />
       </geometry>
     </collision>
@@ -402,19 +384,19 @@
       <geometry>
         <mesh
-          filename="file://$(find carver_description)/meshes/C16_Link.dae" />
-      </geometry>
-      <material
-        name="">
-        <color
-          rgba="0.792156862745098 0.819607843137255 0.933333333333333 1" />
-      </material>
-    </visual>
-    <collision>
-      <origin
-        xyz="0 0 0"
-        rpy="0 0 0" />
-      <geometry>
-        <mesh
-          filename="file://$(find carver_description)/meshes/C16_Link.dae" />
+          filename="file:///$(find carver_description)/meshes/C16_Link.dae" />
+      </geometry>
+      <material
+        name="">
+        <color
+          rgba="0.792156862745098 0.819607843137255 0.933333333333333 1" />
+      </material>
+    </visual>
+    <collision>
+      <origin
+        xyz="0 0 0"
+        rpy="0 0 0" />
+      <geometry>
+        <mesh
+          filename="file:///$(find carver_description)/meshes/C16_Link.dae" />
       </geometry>
     </collision>
@@ -455,5 +437,5 @@
       <geometry>
         <mesh
-          filename="file://$(find carver_description)/meshes/T265_Link.dae" />
+          filename="file:///$(find carver_description)/meshes/T265_Link.dae" />
       </geometry>
       <material
@@ -469,5 +451,5 @@
       <geometry>
         <mesh
-          filename="file://$(find carver_description)/meshes/T265_Link.dae" />
+          filename="file:///$(find carver_description)/meshes/T265_Link.dae" />
       </geometry>
     </collision>
@@ -486,41 +468,4 @@
       xyz="0 0 0" />
   </joint>
-  <!-- <gazebo reference="T265_Link">
-      <material>Gazebo/Yellow</material>
-      <sensor name="sensor_camera" type="depth">
-          <pose>0.0 0.0 0.0 0.0 0.0 0.0</pose>
-          <always_on>1</always_on>
-          <update_rate>10</update_rate>
-          <visualize>1</visualize>
-          <camera name="carver_camera">
-          <image>
-              <format>R8G8B8</format>
-              <width>400</width>
-              <height>400</height>
-          </image>
-          <clip>
-              <near>0.01</near>
-              <far>10.0</far>
-          </clip>
-          </camera>
-          <plugin name="gazebo_ros_depth_camera_sensor" filename="libgazebo_ros_camera.so">
-              <ros>
-                  <namespace>/carver</namespace>
-                  <ros-args>
-                      <remap from="carver_camera/image_raw" to="carver_camera/image"/>
-                      <remap from="carver_camera/image_depth" to="carver_camera/depth/camera_image_depth"/>
-                      <remap from="carver_camera/camera_info" to="carver_camera/camera_info_raw"/>
-                      <remap from="carver_camera/camera_info_depth" to="carver_camera/camera_info_depth"/>
-                      <remap from="carver_camera/points" to="carver_camera/camera_points"/>
-                  </ros-args>
-              </ros>
-              <camera_name>T265</camera_name>
-              <frame_name>T265_Link</frame_name>
-              <hack_baseline>0.07</hack_baseline>
-              <min_depth>0.001</min_depth>
-          </plugin>
-      </sensor>
-  </gazebo>
-   -->
   <link
     name="L515_Link">
@@ -545,5 +490,5 @@
       <geometry>
         <mesh
-          filename="file://$(find carver_description)/meshes/L515_Link.dae" />
+          filename="file:///$(find carver_description)/meshes/L515_Link.dae" />
       </geometry>
       <material
@@ -559,5 +504,5 @@
       <geometry>
         <mesh
-          filename="file://$(find carver_description)/meshes/L515_Link.dae" />
+          filename="file:///$(find carver_description)/meshes/L515_Link.dae" />
       </geometry>
     </collision>
@@ -598,19 +543,19 @@
       <geometry>
         <mesh
-          filename="file://$(find carver_description)/meshes/LD_SICK_Link.dae" />
-      </geometry>
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
File: src/carver_description/urdf/gazebo_control.xacro (robot description, xacro)
@@ -5,5 +5,5 @@
     <plugin filename="libgazebo_ros2_control.so" name="gazebo_ros2_control">
       <!-- Path to your ROS2 control config -->
-      <parameters>$(find carver_description)/config/controllers.yaml</parameters>
+      <parameters>$(find carver_gazebo)/config/controllers.yaml</parameters>
     </plugin>
   </gazebo>
@@ -15,10 +15,10 @@
       </ros>
       <body_name>base_footprint</body_name>
-      <frameName>world</frameName>
+      <frameName>map</frameName>
       <updateRate>100.0</updateRate>
     </plugin>
   </gazebo> -->
   <!-- ROS2 Control block -->
-  <ros2_control name="GazeboSystem" type="system">
+  <ros2_control name="carver_description" type="system">
     <hardware>
       <plugin>gazebo_ros2_control/GazeboSystem</plugin>
@@ -93,4 +93,9 @@
     <maxContacts value="64"/>
   </gazebo> -->
+  <gazebo reference="base_footprint">
+    <minDepth>0.0001</minDepth>
+    <kp value="10000000.0"/>
+    <kd value="1.0"/>
+  </gazebo>
   <gazebo reference="base_link">
     <minDepth>0.0001</minDepth>

File: src/carver_description/urdf/gps.xacro (robot description, xacro)
@@ -23,5 +23,5 @@
       <geometry>
         <mesh
-          filename="file://$(find carver_description)/meshes/GPS_Link.dae" />
+          filename="file:///$(find carver_description)/meshes/GPS_Link.STL" />
       </geometry>
       <material
@@ -37,5 +37,5 @@
       <geometry>
         <mesh
-          filename="file://$(find carver_description)/meshes/GPS_Link.dae" />
+          filename="file:///$(find carver_description)/meshes/GPS_Link.STL" />
       </geometry>
     </collision>

File: src/carver_description/urdf/imu.xacro (robot description, xacro)
@@ -21,5 +21,5 @@
       <geometry>
         <mesh
-          filename="file://$(find carver_description)/meshes/IMU_R_Link.dae" />
+          filename="file:///$(find carver_description)/meshes/IMU_R_Link.STL" />
       </geometry>
       <material name='imu_r_material'>
@@ -37,5 +37,5 @@
       <geometry>
         <mesh
-          filename="file://$(find carver_description)/meshes/IMU_R_Link.dae" />
+          filename="file:///$(find carver_description)/meshes/IMU_R_Link.STL" />
       </geometry>
     </collision>
@@ -74,5 +74,5 @@
       <geometry>
         <mesh
-          filename="file://$(find carver_description)/meshes/IMU_L_Link.dae" />
+          filename="file:///$(find carver_description)/meshes/IMU_L_Link.STL" />
       </geometry>
       <material name='imu_l_material'>
@@ -90,5 +90,5 @@
       <geometry>
         <mesh
-          filename="file://$(find carver_description)/meshes/IMU_L_Link.dae" />
+          filename="file:///$(find carver_description)/meshes/IMU_L_Link.STL" />
       </geometry>
     </collision>

File: src/carver_description/urdf/laser.xacro (robot description, xacro)
@@ -31,5 +31,5 @@
       <geometry>
         <mesh
-          filename="file://$(find carver_description)/meshes/RPLIDAR_LB_Link.STL" />
+          filename="file:///$(find carver_description)/meshes/RPLIDAR_LB_Link.STL" />
       </geometry>
       <material
@@ -45,5 +45,5 @@
       <geometry>
         <mesh
-          filename="file://$(find carver_description)/meshes/RPLIDAR_LB_Link.STL" />
+          filename="file:///$(find carver_description)/meshes/RPLIDAR_LB_Link.STL" />
       </geometry>
     </collision>
@@ -86,5 +86,5 @@
       <geometry>
         <mesh
-          filename="file://$(find carver_description)/meshes/RPLIDAR_RF_Link.STL" />
+          filename="file:///$(find carver_description)/meshes/RPLIDAR_RF_Link.STL" />
       </geometry>
       <material
@@ -100,5 +100,5 @@
       <geometry>
         <mesh
-          filename="file://$(find carver_description)/meshes/RPLIDAR_RF_Link.STL" />
+          filename="file:///$(find carver_description)/meshes/RPLIDAR_RF_Link.STL" />
       </geometry>
     </collision>
@@ -119,73 +119,73 @@
   </joint>
 <!-- /////////////////////////////// -->
-    <gazebo reference="RPLIDAR_LB_Link">
-            <material>Gazebo/Red</material>
-            <sensor name="laser_LB" type="ray">
-            <always_on>true</always_on>
-            <visualize>false</visualize>
-            <update_rate>20</update_rate>
-            <ray>
-                <scan>
-                <horizontal>
-                    <samples>180</samples>
-                    <resolution>0.5</resolution>
-                    <min_angle>-1.91986</min_angle>
-                    <max_angle>0.349066</max_angle>
-                </horizontal>
-                </scan>
-                <range>
-                <min>0.3</min>
-                <max>30.0</max>
-                <resolution>0.01</resolution>
-                </range>
-                <noise>
-                <type>gaussian</type>
-                <mean>0.0</mean>
-                <stddev>0.005</stddev>
-                </noise>
-            </ray>
-            <plugin name="scan_LB" filename="libgazebo_ros_ray_sensor.so">
-                <ros>
-                <remapping>~/out:=scan_LB</remapping>
-                </ros>
-                <output_type>sensor_msgs/LaserScan</output_type>
-                <frame_name>RPLIDAR_LB_Link</frame_name>
-            </plugin>
-            </sensor>
-    </gazebo>
-    <gazebo reference="RPLIDAR_RF_Link">
-            <material>Gazebo/Yellow</material>
-            <sensor name="laser_RF" type="ray">
-            <always_on>true</always_on>
-            <visualize>false</visualize>
-            <update_rate>20</update_rate>
-            <ray>
-                <scan>
-                <horizontal>
-                    <samples>180</samples>
-                    <resolution>0.5</resolution>
-                    <min_angle>-1.91986</min_angle>
-                    <max_angle>0.349066</max_angle>
-               </horizontal>
-                </scan>
-                <range>
-                <min>0.3</min>
-                <max>30.0</max>
-                <resolution>0.01</resolution>
-                </range>
-                <noise>
-                <type>gaussian</type>
-                <mean>0.0</mean>
-                <stddev>0.005</stddev>
-                </noise>
-            </ray>
-            <plugin name="scan_RF" filename="libgazebo_ros_ray_sensor.so">
-                <ros>
-                <remapping>~/out:=scan_RF</remapping>
-                </ros>
-                <output_type>sensor_msgs/LaserScan</output_type>
-                <frame_name>RPLIDAR_RF_Link</frame_name>
-            </plugin>
-            </sensor>
-    </gazebo>
+  <gazebo reference="RPLIDAR_LB_Link">
+          <material>Gazebo/FlatBlack</material>
+          <sensor name="RPLIDAR_LB_Link" type="ray">
+          <always_on>true</always_on>
+          <visualize>false</visualize>
+          <update_rate>12.5</update_rate>
+          <ray>
+              <scan>
+              <horizontal>
+                  <samples>541</samples>
+                  <resolution>1</resolution>
+                  <min_angle>-1.91986</min_angle>
+                  <max_angle>0.349066</max_angle>
+              </horizontal>
+              </scan>
+              <range>
+              <min>0.05</min>
+              <max>29.0</max>
+              <resolution>0.01</resolution>
+              </range>
+              <noise>
+              <type>gaussian</type>
+              <mean>0.0</mean>
+              <stddev>0.01</stddev>
+              </noise>
+          </ray>
+          <plugin name="gazebo_ros_RPLIDAR_LB_Link_controller" filename="libgazebo_ros_ray_sensor.so">
+              <ros>
+              <remapping>~/out:=scan_LB</remapping>
+              </ros>
+              <output_type>sensor_msgs/LaserScan</output_type>
+              <frame_name>RPLIDAR_LB_Link</frame_name>
+          </plugin>
+          </sensor>
+  </gazebo>
+  <gazebo reference="RPLIDAR_RF_Link">
+          <material>Gazebo/FlatBlack</material>
+          <sensor name="RPLIDAR_RF_Link" type="ray">
+          <always_on>true</always_on>
+          <visualize>false</visualize>
+          <update_rate>12.5</update_rate>
+          <ray>
+              <scan>
+              <horizontal>
+                  <samples>541</samples>
+                  <resolution>1</resolution>
+                  <min_angle>-1.91986</min_angle>
+                  <max_angle>0.349066</max_angle>
+              </horizontal>
+              </scan>
+              <range>
+              <min>0.05</min>
+              <max>29.0</max>
+              <resolution>0.01</resolution>
+              </range>
+              <noise>
+              <type>gaussian</type>
+              <mean>0.0</mean>
+              <stddev>0.01</stddev>
+              </noise>
+          </ray>
+          <plugin name="gazebo_ros_RPLIDAR_RF_Link_controller" filename="libgazebo_ros_ray_sensor.so">
+              <ros>
+              <remapping>~/out:=scan_RF</remapping>
+              </ros>
+              <output_type>sensor_msgs/LaserScan</output_type>
+              <frame_name>RPLIDAR_RF_Link</frame_name>
+          </plugin>
+          </sensor>
+  </gazebo>
 </robot>
