Commit message: update much

File: src/carver_description/urdf/carver.xacro (robot description, xacro)
@@ -19,19 +19,19 @@
       <geometry>
         <mesh
-          filename="file:///$(find carver_description)/meshes/base_link.dae" />
-      </geometry>
-      <material
-        name="">
-        <color
-          rgba="0.792156862745098 0.819607843137255 0.933333333333333 1" />
-      </material>
-    </visual>
-    <collision>
-      <origin
-        xyz="0 0 0"
-        rpy="0 0 0" />
-      <geometry>
-        <mesh
-          filename="file:///$(find carver_description)/meshes/base_link.dae" />
+          filename="file:///$(find carver_description)/meshes/base_link.STL" />
+      </geometry>
+      <material
+        name="">
+        <color
+          rgba="0.792156862745098 0.819607843137255 0.933333333333333 1" />
+      </material>
+    </visual>
+    <collision>
+      <origin
+        xyz="0 0 0"
+        rpy="0 0 0" />
+      <geometry>
+        <mesh
+          filename="file:///$(find carver_description)/meshes/base_link.STL" />
       </geometry>
     </collision>
@@ -58,19 +58,19 @@
       <geometry>
         <mesh
-          filename="file:///$(find carver_description)/meshes/front_right_sterring_Link.dae" />
-      </geometry>
-      <material
-        name="">
-        <color
-          rgba="0.792156862745098 0.819607843137255 0.933333333333333 1" />
-      </material>
-    </visual>
-    <collision>
-      <origin
-        xyz="0 0 0"
-        rpy="0 0 0" />
-      <geometry>
-        <mesh
-          filename="file:///$(find carver_description)/meshes/front_right_sterring_Link.dae" />
+          filename="file:///$(find carver_description)/meshes/front_right_sterring_Link.STL" />
+      </geometry>
+      <material
+        name="">
+        <color
+          rgba="0.792156862745098 0.819607843137255 0.933333333333333 1" />
+      </material>
+    </visual>
+    <collision>
+      <origin
+        xyz="0 0 0"
+        rpy="0 0 0" />
+      <geometry>
+        <mesh
+          filename="file:///$(find carver_description)/meshes/front_right_sterring_Link.STL" />
       </geometry>
     </collision>
@@ -111,19 +111,19 @@
       <geometry>
         <mesh
-          filename="file:///$(find carver_description)/meshes/front_right_wheel_Link.dae" />
-      </geometry>
-      <material
-        name="">
-        <color
-          rgba="0.792156862745098 0.819607843137255 0.933333333333333 1" />
-      </material>
-    </visual>
-    <collision>
-      <origin
-        xyz="0 0 0"
-        rpy="0 0 0" />
-      <geometry>
-        <mesh
-          filename="file:///$(find carver_description)/meshes/front_right_wheel_Link.dae" />
+          filename="file:///$(find carver_description)/meshes/front_right_wheel_Link.STL" />
+      </geometry>
+      <material
+        name="">
+        <color
+          rgba="0.792156862745098 0.819607843137255 0.933333333333333 1" />
+      </material>
+    </visual>
+    <collision>
+      <origin
+        xyz="0 0 0"
+        rpy="0 0 0" />
+      <geometry>
+        <mesh
+          filename="file:///$(find carver_description)/meshes/front_right_wheel_Link.STL" />
       </geometry>
     </collision>
@@ -166,19 +166,19 @@
       <geometry>
         <mesh
-          filename="file:///$(find carver_description)/meshes/front_left_sterring_Link.dae" />
-      </geometry>
-      <material
-        name="">
-        <color
-          rgba="0.792156862745098 0.819607843137255 0.933333333333333 1" />
-      </material>
-    </visual>
-    <collision>
-      <origin
-        xyz="0 0 0"
-        rpy="0 0 0" />
-      <geometry>
-        <mesh
-          filename="file:///$(find carver_description)/meshes/front_left_sterring_Link.dae" />
+          filename="file:///$(find carver_description)/meshes/front_left_sterring_Link.STL" />
+      </geometry>
+      <material
+        name="">
+        <color
+          rgba="0.792156862745098 0.819607843137255 0.933333333333333 1" />
+      </material>
+    </visual>
+    <collision>
+      <origin
+        xyz="0 0 0"
+        rpy="0 0 0" />
+      <geometry>
+        <mesh
+          filename="file:///$(find carver_description)/meshes/front_left_sterring_Link.STL" />
       </geometry>
     </collision>
@@ -219,19 +219,19 @@
       <geometry>
         <mesh
-          filename="file:///$(find carver_description)/meshes/front_left_wheel_Link.dae" />
-      </geometry>
-      <material
-        name="">
-        <color
-          rgba="0.792156862745098 0.819607843137255 0.933333333333333 1" />
-      </material>
-    </visual>
-    <collision>
-      <origin
-        xyz="0 0 0"
-        rpy="0 0 0" />
-      <geometry>
-        <mesh
-          filename="file:///$(find carver_description)/meshes/front_left_wheel_Link.dae" />
+          filename="file:///$(find carver_description)/meshes/front_left_wheel_Link.STL" />
+      </geometry>
+      <material
+        name="">
+        <color
+          rgba="0.792156862745098 0.819607843137255 0.933333333333333 1" />
+      </material>
+    </visual>
+    <collision>
+      <origin
+        xyz="0 0 0"
+        rpy="0 0 0" />
+      <geometry>
+        <mesh
+          filename="file:///$(find carver_description)/meshes/front_left_wheel_Link.STL" />
       </geometry>
     </collision>
@@ -273,19 +273,19 @@
       <geometry>
         <mesh
-          filename="file:///$(find carver_description)/meshes/rear_right_wheel_Link.dae" />
-      </geometry>
-      <material
-        name="">
-        <color
-          rgba="0.792156862745098 0.819607843137255 0.933333333333333 1" />
-      </material>
-    </visual>
-    <collision>
-      <origin
-        xyz="0 0 0"
-        rpy="0 0 0" />
-      <geometry>
-        <mesh
-          filename="file:///$(find carver_description)/meshes/rear_right_wheel_Link.dae" />
+          filename="file:///$(find carver_description)/meshes/rear_right_wheel_Link.STL" />
+      </geometry>
+      <material
+        name="">
+        <color
+          rgba="0.792156862745098 0.819607843137255 0.933333333333333 1" />
+      </material>
+    </visual>
+    <collision>
+      <origin
+        xyz="0 0 0"
+        rpy="0 0 0" />
+      <geometry>
+        <mesh
+          filename="file:///$(find carver_description)/meshes/rear_right_wheel_Link.STL" />
       </geometry>
     </collision>
@@ -327,19 +327,19 @@
       <geometry>
         <mesh
-          filename="file:///$(find carver_description)/meshes/rear_left_wheel_Link.dae" />
-      </geometry>
-      <material
-        name="">
-        <color
-          rgba="0.792156862745098 0.819607843137255 0.933333333333333 1" />
-      </material>
-    </visual>
-    <collision>
-      <origin
-        xyz="0 0 0"
-        rpy="0 0 0" />
-      <geometry>
-        <mesh
-          filename="file:///$(find carver_description)/meshes/rear_left_wheel_Link.dae" />
+          filename="file:///$(find carver_description)/meshes/rear_left_wheel_Link.STL" />
+      </geometry>
+      <material
+        name="">
+        <color
+          rgba="0.792156862745098 0.819607843137255 0.933333333333333 1" />
+      </material>
+    </visual>
+    <collision>
+      <origin
+        xyz="0 0 0"
+        rpy="0 0 0" />
+      <geometry>
+        <mesh
+          filename="file:///$(find carver_description)/meshes/rear_left_wheel_Link.STL" />
       </geometry>
     </collision>
@@ -384,19 +384,19 @@
       <geometry>
         <mesh
-          filename="file:///$(find carver_description)/meshes/C16_Link.dae" />
-      </geometry>
-      <material
-        name="">
-        <color
-          rgba="0.792156862745098 0.819607843137255 0.933333333333333 1" />
-      </material>
-    </visual>
-    <collision>
-      <origin
-        xyz="0 0 0"
-        rpy="0 0 0" />
-      <geometry>
-        <mesh
-          filename="file:///$(find carver_description)/meshes/C16_Link.dae" />
+          filename="file:///$(find carver_description)/meshes/C16_Link.STL" />
+      </geometry>
+      <material
+        name="">
+        <color
+          rgba="0.792156862745098 0.819607843137255 0.933333333333333 1" />
+      </material>
+    </visual>
+    <collision>
+      <origin
+        xyz="0 0 0"
+        rpy="0 0 0" />
+      <geometry>
+        <mesh
+          filename="file:///$(find carver_description)/meshes/C16_Link.STL" />
       </geometry>
     </collision>
@@ -437,5 +437,5 @@
       <geometry>
         <mesh
-          filename="file:///$(find carver_description)/meshes/T265_Link.dae" />
+          filename="file:///$(find carver_description)/meshes/T265_Link.STL" />
       </geometry>
       <material
@@ -451,5 +451,5 @@
       <geometry>
         <mesh
-          filename="file:///$(find carver_description)/meshes/T265_Link.dae" />
+          filename="file:///$(find carver_description)/meshes/T265_Link.STL" />
       </geometry>
     </collision>
@@ -490,5 +490,5 @@
       <geometry>
         <mesh
-          filename="file:///$(find carver_description)/meshes/L515_Link.dae" />
+          filename="file:///$(find carver_description)/meshes/L515_Link.STL" />
       </geometry>
       <material
@@ -504,5 +504,5 @@
       <geometry>
         <mesh
-          filename="file:///$(find carver_description)/meshes/L515_Link.dae" />
+          filename="file:///$(find carver_description)/meshes/L515_Link.STL" />
       </geometry>
     </collision>
@@ -543,19 +543,19 @@
       <geometry>
         <mesh
-          filename="file:///$(find carver_description)/meshes/LD_SICK_Link.dae" />
-      </geometry>
-      <material
-        name="">
-        <color
-          rgba="0.792156862745098 0.819607843137255 0.933333333333333 1" />
-      </material>
-    </visual>
-    <collision>
-      <origin
-        xyz="0 0 0"
-        rpy="0 0 0" />
-      <geometry>
-        <mesh
-          filename="file:///$(find carver_description)/meshes/LD_SICK_Link.dae" />
+          filename="file:///$(find carver_description)/meshes/LD_SICK_Link.STL" />
+      </geometry>
+      <material
+        name="">
+        <color
+          rgba="0.792156862745098 0.819607843137255 0.933333333333333 1" />
+      </material>
+    </visual>
+    <collision>
+      <origin
+        xyz="0 0 0"
+        rpy="0 0 0" />
+      <geometry>
+        <mesh
+          filename="file:///$(find carver_description)/meshes/LD_SICK_Link.STL" />
       </geometry>
     </collision>

File: src/carver_description/urdf/gazebo_control.xacro (robot description, xacro)
@@ -18,5 +18,6 @@
       <updateRate>100.0</updateRate>
     </plugin>
-  </gazebo> -->
+  </gazebo>
+ -->
   <!-- ROS2 Control block -->
   <ros2_control name="carver_description" type="system">

File: src/carver_description/urdf/laser.xacro (robot description, xacro)
@@ -122,7 +122,6 @@
           <material>Gazebo/FlatBlack</material>
           <sensor name="RPLIDAR_LB_Link" type="ray">
-          <always_on>true</always_on>
           <visualize>false</visualize>
-          <update_rate>12.5</update_rate>
+          <update_rate>10</update_rate>
           <ray>
               <scan>
@@ -157,7 +156,6 @@
           <material>Gazebo/FlatBlack</material>
           <sensor name="RPLIDAR_RF_Link" type="ray">
-          <always_on>true</always_on>
           <visualize>false</visualize>
-          <update_rate>12.5</update_rate>
+          <update_rate>10</update_rate>
           <ray>
               <scan>
